File: hardware/interface.sch (KiCad schematic (older format))
At the start: 19 parts, among them SW1 DIPSW4_DIP, U4 FXMA108

Commit message: Corrected some colour coding in BOM files.
Still can't get Sueversion ignore to work when using 'svn add'. It works for
'svn status', though. So there's clearly a bug. I've never had this problem
before. Strange.
Changed lines of the file:
@@
 $Descr A4 11693 8268
 encoding utf-8
-Sheet 6 6
+Sheet 2 6
 Title "FREAKDUINO-CHIBI 2.4GHz"
 Date "16 jul 2013"
@@
 $EndComp
 $Comp
-L VSS #PWR052
+L VSS #PWR011
 U 1 1 51E3DBDC
 P 4100 2250
-F 0 "#PWR052" H 4100 2250 30  0001 C CNN
+F 0 "#PWR011" H 4100 2250 30  0001 C CNN
 F 1 "VSS" H 4100 2180 30  0000 C CNN
 F 2 "" H 4100 2250 60  0000 C CNN
@@
 NoConn ~ 4100 3400
 Wire Wire Line
-	2000 2350 2000 2650
-Wire Wire Line
-	2000 2650 2000 3950
-$Comp
-L VSS #PWR053
+	2000 2350 2000 3950
+$Comp
+L VSS #PWR012
 U 1 1 51E3DBEA
 P 3350 4750
-F 0 "#PWR053" H 3350 4750 30  0001 C CNN
+F 0 "#PWR012" H 3350 4750 30  0001 C CNN
 F 1 "VSS" H 3350 4680 30  0000 C CNN
 F 2 "" H 3350 4750 60  0000 C CNN
@@
 $EndComp
 Wire Wire Line
-	3350 4150 3350 4600
-Wire Wire Line
-	3350 4600 3350 4750
+	3350 4150 3350 4750
 Wire Wire Line
 	3550 4600 3550 4150
 Wire Wire Line
-	2000 4600 3350 4600
-Wire Wire Line
-	3350 4600 3550 4600
+	2000 4600 3550 4600
 Connection ~ 3350 4600
 Wire Wire Line
@@
 $EndComp
 $Comp
-L VSS #PWR054
+L VSS #PWR013
 U 1 1 51E3DC0E
 P 2450 2250
-F 0 "#PWR054" H 2450 2250 30  0001 C CNN
+F 0 "#PWR013" H 2450 2250 30  0001 C CNN
 F 1 "VSS" H 2450 2180 30  0000 C CNN
 F 2 "" H 2450 2250 60  0000 C CNN
@@
 	4100 3300 5100 3300
 $Comp
-L VCC5 #PWR055
+L VCC5 #PWR014
 U 1 1 51E3DC24
 P 4100 1450
-F 0 "#PWR055" H 4100 1590 20  0001 C CNN
+F 0 "#PWR014" H 4100 1590 20  0001 C CNN
 F 1 "VCC5" H 4100 1560 30  0000 C CNN
 F 2 "" H 4100 1450 60  0000 C CNN
@@
 $EndComp
 $Comp
-L VCC5 #PWR056
+L VCC5 #PWR015
 U 1 1 51E3DC2A
 P 3550 1450
-F 0 "#PWR056" H 3550 1590 20  0001 C CNN
+F 0 "#PWR015" H 3550 1590 20  0001 C CNN
 F 1 "VCC5" H 3550 1560 30  0000 C CNN
 F 2 "" H 3550 1450 60  0000 C CNN
@@
 $EndComp
 $Comp
-L VCC3 #PWR057
+L VCC3 #PWR016
 U 1 1 51E3DC30
 P 3350 1600
-F 0 "#PWR057" H 3350 1740 20  0001 C CNN
+F 0 "#PWR016" H 3350 1740 20  0001 C CNN
 F 1 "VCC3" H 3350 1710 30  0000 C CNN
 F 2 "" H 3350 1600 60  0000 C CNN
@@
 $EndComp
 $Comp
-L VCC3 #PWR058
+L VCC3 #PWR017
 U 1 1 51E3DC36
 P 2450 1600
-F 0 "#PWR058" H 2450 1740 20  0001 C CNN
+F 0 "#PWR017" H 2450 1740 20  0001 C CNN
 F 1 "VCC3" H 2450 1710 30  0000 C CNN
 F 2 "" H 2450 1600 60  0000 C CNN
@@
 $EndComp
 $Comp
-L VCC3 #PWR059
+L VCC3 #PWR018
 U 1 1 51E3DC3C
 P 2000 1600
-F 0 "#PWR059" H 2000 1740 20  0001 C CNN
+F 0 "#PWR018" H 2000 1740 20  0001 C CNN
 F 1 "VCC3" H 2000 1710 30  0000 C CNN
 F 2 "" H 2000 1600 60  0000 C CNN
@@
 	5950 4350 5950 5000
 $Comp
-L VSS #PWR060
+L VSS #PWR019
 U 1 1 51E3E179
 P 5950 5700
-F 0 "#PWR060" H 5950 5700 30  0001 C CNN
+F 0 "#PWR019" H 5950 5700 30  0001 C CNN
 F 1 "VSS" H 5950 5630 30  0000 C CNN
 F 2 "" H 5950 5700 60  0000 C CNN
@@
 $EndComp
 $Comp
-L VSS #PWR061
+L VSS #PWR020
 U 1 1 51E3E17F
 P 6450 5700
-F 0 "#PWR061" H 6450 5700 30  0001 C CNN
+F 0 "#PWR020" H 6450 5700 30  0001 C CNN
 F 1 "VSS" H 6450 5630 30  0000 C CNN
 F 2 "" H 6450 5700 60  0000 C CNN
@@
 VCC3_LED
 $Comp
-L VCC3 #PWR062
+L VCC3 #PWR021
 U 1 1 51E3E18C
 P 6450 2300
-F 0 "#PWR062" H 6450 2440 20  0001 C CNN
+F 0 "#PWR021" H 6450 2440 20  0001 C CNN
 F 1 "VCC3" H 6450 2410 30  0000 C CNN
 F 2 "" H 6450 2300 60  0000 C CNN
@@
 $EndComp
 $Comp
-L VCC5 #PWR063
+L VCC5 #PWR022
 U 1 1 51E3E192
 P 6250 2100
-F 0 "#PWR063" H 6250 2240 20  0001 C CNN
+F 0 "#PWR022" H 6250 2240 20  0001 C CNN
 F 1 "VCC5" H 6250 2210 30  0000 C CNN
 F 2 "" H 6250 2100 60  0000 C CNN
@@
 	4250 6950 4250 7250
 $Comp
-L VSS #PWR064
+L VSS #PWR023
 U 1 1 51E3E429
 P 4250 7250
-F 0 "#PWR064" H 4250 7250 30  0001 C CNN
+F 0 "#PWR023" H 4250 7250 30  0001 C CNN
 F 1 "VSS" H 4250 7180 30  0000 C CNN
 F 2 "" H 4250 7250 60  0000 C CNN
@@
 ISP CONNECTOR
 $Comp
-L VCC5 #PWR065
+L VCC5 #PWR024
 U 1 1 51E3E434
 P 4250 6400
-F 0 "#PWR065" H 4250 6540 20  0001 C CNN
+F 0 "#PWR024" H 4250 6540 20  0001 C CNN
 F 1 "VCC5" H 4250 6510 30  0000 C CNN
 F 2 "" H 4250 6400 60  0000 C CNN
@@
 $EndComp
 $Comp
-L VSS #PWR066
+L VSS #PWR025
 U 1 1 51E3E736
 P 7550 6450
-F 0 "#PWR066" H 7550 6450 30  0001 C CNN
+F 0 "#PWR025" H 7550 6450 30  0001 C CNN
 F 1 "VSS" H 7550 6380 30  0000 C CNN
 F 2 "" H 7550 6450 60  0000 C CNN
@@
 PB5/SCLK
 Wire Wire Line
-	9400 3800 9650 3800
-Wire Wire Line
-	9650 3800 9800 3800
-Wire Wire Line
-	9400 3900 9750 3900
-Wire Wire Line
-	9750 3900 9800 3900
+	9400 3800 9800 3800
+Wire Wire Line
+	9400 3900 9800 3900
 Wire Wire Line
 	9800 4000 9400 4000
@@
 	9650 5600 9650 5850
 $Comp
-L VSS #PWR067
+L VSS #PWR026
 U 1 1 51E3E76E
 P 9650 5850
-F 0 "#PWR067" H 9650 5850 30  0001 C CNN
+F 0 "#PWR026" H 9650 5850 30  0001 C CNN
 F 1 "VSS" H 9650 5780 30  0000 C CNN
 F 2 "" H 9650 5850 60  0000 C CNN
@@
 	9100 2100 9100 1000
 $Comp
-L VSS #PWR068
+L VSS #PWR027
 U 1 1 51E3E798
 P 9650 2300
-F 0 "#PWR068" H 9650 2300 30  0001 C CNN
+F 0 "#PWR027" H 9650 2300 30  0001 C CNN
 F 1 "VSS" H 9650 2230 30  0000 C CNN
 F 2 "" H 9650 2300 60  0000 C CNN
@@
 	9750 1900 9650 1900
 Wire Wire Line
-	9650 1900 9650 2000
-Wire Wire Line
-	9650 2000 9650 2300
+	9650 1900 9650 2300
 Wire Wire Line
 	9750 2000 9650 2000
 Connection ~ 9650 2000
 $Comp
-L VCC5 #PWR069
+L VCC5 #PWR028
 U 1 1 51E3E7A3
 P 9400 1100
-F 0 "#PWR069" H 9400 1240 20  0001 C CNN
+F 0 "#PWR028" H 9400 1240 20  0001 C CNN
 F 1 "VCC5" H 9400 1210 30  0000 C CNN
 F 2 "" H 9400 1100 60  0000 C CNN
@@
 $EndComp
 $Comp
-L VCC3 #PWR070
+L VCC3 #PWR029
 U 1 1 51E3E7A9
 P 9650 1200
-F 0 "#PWR070" H 9650 1340 20  0001 C CNN
+F 0 "#PWR029" H 9650 1340 20  0001 C CNN
 F 1 "VCC3" H 9650 1310 30  0000 C CNN
 F 2 "" H 9650 1200 60  0000 C CNN
@@
 $EndComp
 $Comp
-L VCC_IN #PWR071
+L VCC_IN #PWR030
 U 1 1 51E3E7C7
 P 9100 1000
-F 0 "#PWR071" H 9100 1140 20  0001 C CNN
+F 0 "#PWR030" H 9100 1140 20  0001 C CNN
 F 1 "VCC_IN" H 9100 1110 30  0000 C CNN
 F 2 "" H 9100 1000 60  0000 C CNN
